Commit message: Changes for adding panda emika into planning environment. Pickup box currently not being generated correctly.

File: exercises/Optimization_Based_Planning/solution_ws/src/pick_and_place_support/include/robot_description/oak_d.xacro (robot description, xacro)
@@ -1,4 +1,4 @@
 <?xml version="1.0" encoding="utf-8"?>
-<robot xmlns:xacro="http://www.ros.org/wiki/xacro" name="suction_ee">
+<robot xmlns:xacro="http://www.ros.org/wiki/xacro" name="panda">
   <!-- safety_distance: Minimum safety distance in [m] by which the collision volumes are expanded and which is enforced during robot motions -->
   <xacro:macro name="oak_d" params="connected_to:='' rpy:='0 0 0' xyz:='0 0 0' safety_distance:=0 id:='oak_d_default'">

File: exercises/Optimization_Based_Planning/solution_ws/src/pick_and_place_support/include/robot_description/panda_arm.urdf.xacro (robot description, xacro)
@@ -1,4 +1,6 @@
 <?xml version='1.0' encoding='utf-8'?>
 <robot xmlns:xacro="http://www.ros.org/wiki/xacro" name="panda">
+  <link name="world"/>
+  <link name="base_link"/>
   <xacro:arg name="arm_id" default="panda"/> <!-- Name of this panda -->
   <xacro:arg name="suction_ee" default="true"/>
@@ -6,6 +8,20 @@
   <xacro:arg name="use_fake_hardware" default="false"/>
   <xacro:arg name="fake_sensor_commands" default="false"/>
+  <!-- Include workcell (creates joint from world to workcell_base)-->
+  <xacro:include filename="$(find pick_and_place_support)/urdf/environment.xacro"/>
+  <xacro:workcell parent_link="world" >
+    <origin xyz="0.0 0.0 0.77153" rpy="0 0 0"/>
+  </xacro:workcell >
+  <xacro:cabinet id="1" parent_link="workcell_base" >
+    <origin rpy="0 0 0" xyz="-0.3048 1.016 0.771525"/>
+  </xacro:cabinet >
+  <!-- Create joints -->
+  <joint name="workcell_base_to_base" type="fixed">
+    <parent link="workcell_base"/>
+    <child link="base_link"/>
+    <origin xyz="0 -0.0381 0.00953" rpy="0 0 1.5708"/>
+  </joint>
   <xacro:include filename="$(find pick_and_place_support)/include/robot_description/panda_arm.xacro"/>
-  <xacro:panda_arm arm_id="$(arg arm_id)" safety_distance="0.01"/>
+  <xacro:panda_arm arm_id="$(arg arm_id)" connected_to="base_link" safety_distance="0.01"/>
   <xacro:if value="$(arg suction_ee)">
     <xacro:include filename="$(find pick_and_place_support)/include/robot_description/suction_ee.xacro"/>

File: exercises/Optimization_Based_Planning/solution_ws/src/pick_and_place_support/include/robot_semantic_description/panda_arm.srdf.xacro (robot description, xacro)
@@ -1,4 +1,16 @@
 <?xml version='1.0' encoding='utf-8'?>
 <robot xmlns:xacro="http://www.ros.org/wiki/xacro" name="panda">
+  <group name="Manipulator">
+    <chain base_link="base_link" tip_link="panda_ee_tcp" />
+  </group>
+  <group_state name="AllZero" group="Manipulator">
+        <joint name="panda_joint1" value="0" />
+        <joint name="panda_joint2" value="0" />
+        <joint name="panda_joint3" value="0" />
+        <joint name="panda_joint4" value="0" />
+        <joint name="panda_joint5" value="0" />
+        <joint name="panda_joint6" value="0" />
+        <joint name="panda_joint7" value="0" />
+    </group_state>
   <xacro:arg name="arm_id" default="panda"/> <!-- Name of this panda -->
   <xacro:arg name="suction_ee" default="true"/> <!-- Should a franka_gripper be mounted at the flange? (Currently does not work without it) -->
